Commit message: Gaits optimized.

File: src/arboc_description/urdf/arboc.urdf (robot description, URDF)
Before this commit: robot arboc, 9 links, 8 joints
Joints:
- joint joint_01: limit lower=-1.57 upper=1.57 effort=15.0 velocity=2.0 -> lower=${-5*PI/12} upper=${5*PI/12} effort=7.0 velocity=2.0
- joint joint_02: limit lower=-1.57 upper=1.57 effort=15.0 velocity=2.0 -> lower=${-5*PI/12} upper=${5*PI/12} effort=7.0 velocity=2.0
- joint joint_03: limit lower=-1.57 upper=1.57 effort=15.0 velocity=2.0 -> lower=${-5*PI/12} upper=${5*PI/12} effort=7.0 velocity=2.0
- joint joint_04: limit lower=-1.57 upper=1.57 effort=15.0 velocity=2.0 -> lower=${-5*PI/12} upper=${5*PI/12} effort=7.0 velocity=2.0
- joint joint_05: limit lower=-1.57 upper=1.57 effort=15.0 velocity=2.0 -> lower=${-5*PI/12} upper=${5*PI/12} effort=7.0 velocity=2.0
- joint joint_06: limit lower=-1.57 upper=1.57 effort=15.0 velocity=2.0 -> lower=${-5*PI/12} upper=${5*PI/12} effort=7.0 velocity=2.0
- joint joint_07: limit lower=-1.57 upper=1.57 effort=15.0 velocity=2.0 -> lower=${-5*PI/12} upper=${5*PI/12} effort=7.0 velocity=2.0
